Commit message: add head extended link

File: protomotions/data/assets/urdf/t1.urdf (robot description, URDF)
Before this commit: robot T1, 28 links, 27 joints
Links:
- added link head_link; visual sphere radius=0.0001
Joints:
- added joint head: type fixed, parent H2, child head_link, origin xyz=0.01 0 0.11 rpy=0 0 0
